File: jscarpa/onboad.kicad_sch (KiCad schematic)
At the start: 11 parts, among them J1 Conn_01x02_Socket, J2 Conn_01x02_Socket, U1 ACS711xLCTR-12AB, U2 mcp6546-e/p

Commit message: Onboarding: Fixed footprint and symbol library directories.
Parts:
- U2: footprint Package_DIP:DIP-8_W7.62mm -> kicad_models:PDIP8_300MC_MCH
